File: BatteryCo/BatteryCo.kicad_sch (KiCad schematic)
At the start: 135 parts, among them J1 Micro_SD_Card_Det2, J10 RJ45_LED_Shielded, J11 RJ45_LED_Shielded, J12 Conn_01x01, J14 Conn_02x05_Counter_Clockwise, J15 Conn_02x05_Odd_Even, J16 Conn_01x03, J19 Conn_01x04, J2 Conn_01x03, J20 Conn_01x04, J22 I2C_BUS0, J24 Conn_02x05_Odd_Even, J3 USB_C_Receptacle_USB2.0_16P, J4 Conn_01x01, J5 Conn_01x01, J7 Conn_01x01, J8 Conn_01x01, J9 Conn_01x01, Q1 IRLZ44SPbF, Q3 AO3400A, Q4 AON6411, Q5 AON6411, Q6 AO3400A, SW1 SW_Push, SW2 SW_Push, SW3 SW_Push, U1 ESP32-S3-WROOM-1, U10 QRE1113GR / ITR8307, U11 QRE1113GR / ITR8307, U12 QRE1113GR / ITR8307, U13 QRE1113GR / ITR8307, U14 QRE1113GR / ITR8307, U15 CA-IS13092VW, U2 QRE1113GR / ITR8307, U3 QRE1113GR / ITR8307, U4 INA228, U5 TPS5430DDA, U6 MCP4728, U7 AMS1117-3.3, U8 SP3485EN, U9 L78M05ABDT-TR

Commit message: Commit before changing to isolated measurement
Parts:
- U5: LCSC Part # (none) -> C9864
Changed lines of the file:
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@@
 (kicad_sch
-	(version 20231120)
+	(version 20250114)
 	(generator "eeschema")
-	(generator_version "8.0")
+	(generator_version "9.0")
 	(paper "B")
+	(rectangle
+		(start 62.23 227.33)
+		(end 106.68 261.62)
+		(stroke
+			(width 0.635)
+			(type dot)
+		)
+		(fill
+			(type none)
+		)
+	)
+	(rectangle
+		(start 15.24 189.23)
+		(end 59.69 223.52)
+		(stroke
+			(width 0.635)
+			(type dot)
+		)
+		(fill
+			(type none)
+		)
+	)
+	(rectangle
+		(start 308.61 161.29)
+		(end 412.75 228.6)
+		(stroke
+			(width 0.635)
+			(type dot)
+		)
+		(fill
+			(type none)
+		)
+	)
+	(rectangle
+		(start 15.24 227.33)
+		(end 59.69 261.62)
+		(stroke
+			(width 0.635)
+			(type dot)
+		)
+		(fill
+			(type none)
+		)
+	)
+	(rectangle
+		(start 62.23 189.23)
+		(end 106.68 223.52)
+		(stroke
+			(width 0.635)
+			(type dot)
+		)
+		(fill
+			(type none)
+		)
+	)
+	(rectangle
+		(start 228.6 196.85)
+		(end 300.99 261.62)
+		(stroke
+			(width 0.635)
+			(type dot)
+		)
+		(fill
+			(type none)
+		)
+	)
+	(rectangle
+		(start 110.49 189.23)
+		(end 222.25 261.62)
+		(stroke
+			(width 0.635)
+			(type dot)
+		)
+		(fill
+			(type none)
+		)
+	)
+	(text "Battery ID\n"
+		(exclude_from_sim no)
+		(at 38.862 234.188 0)
+		(effects
+			(font
+				(size 2.54 2.54)
+				(thickness 0.508)
+				(bold yes)
+			)
+		)
+	)
+	(text "SD CARD"
+		(exclude_from_sim no)
+		(at 124.714 196.342 0)
+		(effects
+			(font
+				(size 2.54 2.54)
+				(thickness 0.508)
+				(bold yes)
+			)
+		)
+	)
+	(text "ESP USB Port"
+		(exclude_from_sim no)
+		(at 263.144 201.676 0)
+		(effects
+			(font
+				(size 2.54 2.54)
+				(thickness 0.508)
+				(bold yes)
+			)
+		)
+	)
+	(text "I2C Pullups"
+		(exclude_from_sim no)
+		(at 38.862 196.088 0)
+		(effects
+			(font
+				(size 2.54 2.54)
+				(thickness 0.508)
+				(bold yes)
+			)
+		)
+	)
+	(text "HiLetgo Ethernet"
+		(exclude_from_sim no)
+		(at 85.852 196.088 0)
+		(effects
+			(font
+				(size 2.54 2.54)
+				(thickness 0.508)
+				(bold yes)
+			)
+		)
+	)
+	(text "VOLTAGE REGULATOR 3.3V\n "
+		(exclude_from_sim no)
+		(at 336.296 168.91 0)
+		(effects
+			(font
+				(size 2.54 2.54)
+				(thickness 0.508)
+				(bold yes)
+			)
+		)
+	)
+	(text "LCD I2C Interface"
+		(exclude_from_sim no)
+		(at 85.852 234.188 0)
+		(effects
+			(font
+				(size 2.54 2.54)
+				(thickness 0.508)
+				(bold yes)
+			)
+		)
+	)
 	(junction
 		(at 285.75 214.63)
@@
 		)
 	)
-	(rectangle
-		(start 62.23 227.33)
-		(end 106.68 261.62)
-		(stroke
-			(width 0.635)
-			(type dot)
-		)
-		(fill
-			(type none)
-		)
-	)
-	(rectangle
-		(start 15.24 189.23)
-		(end 59.69 223.52)
-		(stroke
-			(width 0.635)
-			(type dot)
-		)
-		(fill
-			(type none)
-		)
-	)
-	(rectangle
-		(start 308.61 161.29)
-		(end 412.75 228.6)
-		(stroke
-			(width 0.635)
-			(type dot)
-		)
-		(fill
-			(type none)
-		)
-	)
-	(rectangle
-		(start 15.24 227.33)
-		(end 59.69 261.62)
-		(stroke
-			(width 0.635)
-			(type dot)
-		)
-		(fill
-			(type none)
-		)
-	)
-	(rectangle
-		(start 62.23 189.23)
-		(end 106.68 223.52)
-		(stroke
-			(width 0.635)
-			(type dot)
-		)
-		(fill
-			(type none)
-		)
-	)
-	(rectangle
-		(start 228.6 196.85)
-		(end 300.99 261.62)
-		(stroke
-			(width 0.635)
-			(type dot)
-		)
-		(fill
-			(type none)
-		)
-	)
-	(rectangle
-		(start 110.49 189.23)
-		(end 222.25 261.62)
-		(stroke
-			(width 0.635)
-			(type dot)
-		)
-		(fill
-			(type none)
-		)
-	)
-	(text "Battery ID\n"
-		(exclude_from_sim no)
-		(at 38.862 234.188 0)
-		(effects
-			(font
-				(size 2.54 2.54)
-				(thickness 0.508)
-				(bold yes)
-			)
-		)
-	)
-	(text "SD CARD"
-		(exclude_from_sim no)
-		(at 124.714 196.342 0)
-		(effects
-			(font
-				(size 2.54 2.54)
-				(thickness 0.508)
-				(bold yes)
-			)
-		)
-	)
-	(text "ESP USB Port"
-		(exclude_from_sim no)
-		(at 263.144 201.676 0)
-		(effects
-			(font
-				(size 2.54 2.54)
-				(thickness 0.508)
-				(bold yes)
-			)
-		)
-	)
-	(text "I2C Pullups"
-		(exclude_from_sim no)
-		(at 38.862 196.088 0)
-		(effects
-			(font
-				(size 2.54 2.54)
-				(thickness 0.508)
-				(bold yes)
-			)
-		)
-	)
-	(text "HiLetgo Ethernet"
-		(exclude_from_sim no)
-		(at 85.852 196.088 0)
-		(effects
-			(font
-				(size 2.54 2.54)
-				(thickness 0.508)
-				(bold yes)
-			)
-		)
-	)
-	(text "VOLTAGE REGULATOR 3.3V\n "
-		(exclude_from_sim no)
-		(at 336.296 168.91 0)
-		(effects
-			(font
-				(size 2.54 2.54)
-				(thickness 0.508)
-				(bold yes)
-			)
-		)
-	)
-	(text "LCD I2C Interface"
-		(exclude_from_sim no)
-		(at 85.852 234.188 0)
-		(effects
-			(font
-				(size 2.54 2.54)
-				(thickness 0.508)
-				(bold yes)
-			)
-		)
-	)
 	(global_label "LED_ON"
 		(shape input)
@@
 			)
 		)
+		(property "LCSC Part #" "C9864"
+			(at 328.93 104.14 0)
+			(effects
+				(font
+					(size 1.27 1.27)
+				)
+				(hide yes)
+			)
+		)
 		(pin "5"
 		)
@@
 		)
 	)
+	(embedded_fonts no)
 )
